File: up-hdmi.brd (EAGLE design)
At the start: 20 x 24 mm, 2 parts, among them CON1 HDMI_MALE, CON2 HDMI_MALE

Commit message: Fix length
Parts:
- moved CON2 0.50 mm to (10.0, 19.5)
Routing:
- net N$9: track 12.4 -> 12.9 mm
- net N$7: track 13.0 -> 13.5 mm
- net N$6: track 38.3 -> 38.8 mm
- net N$4: track 38.1 -> 38.6 mm
- net N$3: track 18.0 -> 18.5 mm
- net N$2: track 11.4 -> 11.9 mm
- net N$18: track 28.7 -> 29.2 mm
- net N$17: track 14.9 -> 15.4 mm
- net N$16: track 34.2 -> 34.7 mm
- net N$15: track 16.8 -> 17.3 mm
- net N$14: track 24.6 -> 25.1 mm
- net N$13: track 14.0 -> 14.5 mm
- net N$12: track 27.8 -> 28.3 mm
- net N$10: track 37.2 -> 37.7 mm
- net N$1: track 18.2 -> 18.7 mm
Other:
- board size 20 x 24 mm -> 19 x 24.5 mm
- board text added: "UP-Board | HDMI"
- board text added: "at-wat.tokyo"
